Commit message: Rebuilt the ego racecar so the laser scan originates from the front instead of the back. This was done by shifting all the objects which are jointed to the base_link such that the base_link would be at the front of the car instead of the back (the laser is attached to the base_link's origin point).

File: install/f1tenth_gym_ros/share/f1tenth_gym_ros/launch/ego_racecar.xacro (robot description, xacro)
@@ -8,5 +8,5 @@
   <xacro:property name="wheel_radius" value="0.0508" />
   <xacro:property name="wheel_length" value="0.0381" />
-  <xacro:property name="laser_distance_from_base_link" value="0.275" />
+  <xacro:property name="laser_distance_from_base_link" value="0.0" />
   <xacro:property name="laser_height" value="0.05" />
   <xacro:property name="laser_radius" value="0.026" />
@@ -20,5 +20,5 @@
   <link name="${car_name}/base_link">
     <visual>
-      <origin xyz="${wheelbase/2} 0 ${ground_offset+height/2}"/>
+      <origin xyz="-${wheelbase/2} 0 ${ground_offset+height/2}"/>
       <geometry>
         <box size="${wheelbase} ${width} ${height}"/>
@@ -43,5 +43,5 @@
     <parent link="${car_name}/base_link"/>
     <child link="${car_name}/back_left_wheel"/>
-    <origin xyz="0 ${(wheel_length+width)/2} ${wheel_radius}"/>
+    <origin xyz="-${wheelbase} ${(wheel_length+width)/2} ${wheel_radius}"/>
   </joint>
   <link name="${car_name}/back_left_wheel">
@@ -57,5 +57,5 @@
     <parent link="${car_name}/base_link"/>
     <child link="${car_name}/back_right_wheel"/>
-    <origin xyz="0 ${-(wheel_length+width)/2} ${wheel_radius}"/>
+    <origin xyz="-${wheelbase} ${-(wheel_length+width)/2} ${wheel_radius}"/>
   </joint>
   <link name="${car_name}/back_right_wheel">
@@ -71,5 +71,5 @@
     <parent link="${car_name}/base_link"/>
     <child link="${car_name}/front_left_hinge"/>
-    <origin xyz="${wheelbase} ${(wheel_length+width)/2} ${wheel_radius}"/>
+    <origin xyz="0 ${(wheel_length+width)/2} ${wheel_radius}"/>
   </joint>
   <link name="${car_name}/front_left_hinge"/>
@@ -90,5 +90,5 @@
     <parent link="${car_name}/base_link"/>
     <child link="${car_name}/front_right_hinge"/>
-    <origin xyz="${wheelbase} ${-(wheel_length+width)/2} ${wheel_radius}"/>
+    <origin xyz="0 ${-(wheel_length+width)/2} ${wheel_radius}"/>
   </joint>
   <link name="${car_name}/front_right_hinge"/>
@@ -106,3 +106,13 @@
     </visual>
   </link>
+  <!-- <link name="${car_name}/laser">
+    <visual>
+      <origin xyz="0 5 0"/>
+    </visual>
+  </link>
+  <joint name="base_link_to_laser" type="fixed">
+    <parent link="${car_name}/base_link"/>
+    <child link="${car_name}/laser"/>
+    <origin xyz="0 5 0"/>
+  </joint> -->
 </robot>

File: sim_ws/src/f1tenth_gym_ros/launch/ego_racecar.xacro (robot description, xacro)
@@ -8,5 +8,5 @@
   <xacro:property name="wheel_radius" value="0.0508" />
   <xacro:property name="wheel_length" value="0.0381" />
-  <xacro:property name="laser_distance_from_base_link" value="0.275" />
+  <!-- <xacro:property name="laser_distance_from_base_link" value="0.275" /> -->
   <xacro:property name="laser_height" value="0.05" />
   <xacro:property name="laser_radius" value="0.026" />
@@ -20,5 +20,5 @@
   <link name="${car_name}/base_link">
     <visual>
-      <origin xyz="${wheelbase/2} 0 ${ground_offset+height/2}"/>
+      <origin xyz="-${wheelbase/2} 0 ${ground_offset+height/2}"/>
       <geometry>
         <box size="${wheelbase} ${width} ${height}"/>
@@ -30,5 +30,5 @@
     <parent link="${car_name}/base_link"/>
     <child link="${car_name}/laser_model"/>
-    <origin xyz="${laser_distance_from_base_link} 0 ${ground_offset+height+(laser_height/2)}"/>
+    <origin xyz="0 0 ${ground_offset+height+(laser_height/2)}"/>
   </joint>
   <link name="${car_name}/laser_model">
@@ -43,5 +43,5 @@
     <parent link="${car_name}/base_link"/>
     <child link="${car_name}/back_left_wheel"/>
-    <origin xyz="0 ${(wheel_length+width)/2} ${wheel_radius}"/>
+    <origin xyz="-${wheelbase} ${(wheel_length+width)/2} ${wheel_radius}"/>
   </joint>
   <link name="${car_name}/back_left_wheel">
@@ -57,5 +57,5 @@
     <parent link="${car_name}/base_link"/>
     <child link="${car_name}/back_right_wheel"/>
-    <origin xyz="0 ${-(wheel_length+width)/2} ${wheel_radius}"/>
+    <origin xyz="-${wheelbase} ${-(wheel_length+width)/2} ${wheel_radius}"/>
   </joint>
   <link name="${car_name}/back_right_wheel">
@@ -71,5 +71,5 @@
     <parent link="${car_name}/base_link"/>
     <child link="${car_name}/front_left_hinge"/>
-    <origin xyz="${wheelbase} ${(wheel_length+width)/2} ${wheel_radius}"/>
+    <origin xyz="0 ${(wheel_length+width)/2} ${wheel_radius}"/>
   </joint>
   <link name="${car_name}/front_left_hinge"/>
@@ -90,5 +90,5 @@
     <parent link="${car_name}/base_link"/>
     <child link="${car_name}/front_right_hinge"/>
-    <origin xyz="${wheelbase} ${-(wheel_length+width)/2} ${wheel_radius}"/>
+    <origin xyz="0 ${-(wheel_length+width)/2} ${wheel_radius}"/>
   </joint>
   <link name="${car_name}/front_right_hinge"/>

Commit message: Refactored 'reactive_node' script by putting reused code into separate module scripts.

File: install/f1tenth_gym_ros/share/f1tenth_gym_ros/launch/ego_racecar.xacro (robot description, xacro)
@@ -8,5 +8,5 @@
   <xacro:property name="wheel_radius" value="0.0508" />
   <xacro:property name="wheel_length" value="0.0381" />
-  <xacro:property name="laser_distance_from_base_link" value="0.0" />
+  <!-- <xacro:property name="laser_distance_from_base_link" value="0.275" /> -->
   <xacro:property name="laser_height" value="0.05" />
   <xacro:property name="laser_radius" value="0.026" />
@@ -30,5 +30,5 @@
     <parent link="${car_name}/base_link"/>
     <child link="${car_name}/laser_model"/>
-    <origin xyz="${laser_distance_from_base_link} 0 ${ground_offset+height+(laser_height/2)}"/>
+    <origin xyz="0 0 ${ground_offset+height+(laser_height/2)}"/>
   </joint>
   <link name="${car_name}/laser_model">
@@ -106,13 +106,3 @@
     </visual>
   </link>
-  <!-- <link name="${car_name}/laser">
-    <visual>
-      <origin xyz="0 5 0"/>
-    </visual>
-  </link>
-  <joint name="base_link_to_laser" type="fixed">
-    <parent link="${car_name}/base_link"/>
-    <child link="${car_name}/laser"/>
-    <origin xyz="0 5 0"/>
-  </joint> -->
 </robot>
